File: calculator_interface/keypad.kicad_sch (KiCad schematic)
At the start: 22 parts, among them J2 Conn_02x20_TI30XA, J3 Conn_01x10_TI30XA, Q1 2N7000, Q10 2N7000, Q11 2N7000, Q12 2N7000, Q13 2N7000, Q14 2N7000, Q15 2N7000, Q16 2N7000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

Commit message: add mounting holes
Parts:
- renumbered J3 to J7
Changed lines of the file:
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@@
   (symbol (lib_id "power:GND") (at 48.26 31.75 270) (unit 1)
     (in_bom yes) (on_board yes) (fields_autoplaced)
-    (property "Reference" "#PWR047" (id 0) (at 41.91 31.75 0)
+    (property "Reference" "#PWR051" (id 0) (at 41.91 31.75 0)
       (effects (font (size 1.27 1.27)) hide)
     )
@@
   (symbol (lib_id "custom_connetors:Conn_01x10_TI30XA") (at 97.79 41.91 0) (unit 1)
     (in_bom yes) (on_board yes)
-    (property "Reference" "J3" (id 0) (at 90.17 49.53 0)
+    (property "Reference" "J7" (id 0) (at 90.17 49.53 0)
       (effects (font (size 1.27 1.27)) (justify left))
     )
@@
   (symbol (lib_id "power:+3V3") (at 55.88 82.55 0) (unit 1)
     (in_bom yes) (on_board yes) (fields_autoplaced)
-    (property "Reference" "#PWR051" (id 0) (at 55.88 86.36 0)
+    (property "Reference" "#PWR055" (id 0) (at 55.88 86.36 0)
       (effects (font (size 1.27 1.27)) hide)
     )
@@
   (symbol (lib_id "power:GND") (at 137.16 156.21 0) (unit 1)
     (in_bom yes) (on_board yes) (fields_autoplaced)
-    (property "Reference" "#PWR053" (id 0) (at 137.16 162.56 0)
+    (property "Reference" "#PWR057" (id 0) (at 137.16 162.56 0)
       (effects (font (size 1.27 1.27)) hide)
     )
@@
   (symbol (lib_id "power:+3V3") (at 55.88 24.13 0) (unit 1)
     (in_bom yes) (on_board yes) (fields_autoplaced)
-    (property "Reference" "#PWR049" (id 0) (at 55.88 27.94 0)
+    (property "Reference" "#PWR053" (id 0) (at 55.88 27.94 0)
       (effects (font (size 1.27 1.27)) hide)
     )
@@
   (symbol (lib_id "power:GND") (at 48.26 90.17 270) (unit 1)
     (in_bom yes) (on_board yes) (fields_autoplaced)
-    (property "Reference" "#PWR048" (id 0) (at 41.91 90.17 0)
+    (property "Reference" "#PWR052" (id 0) (at 41.91 90.17 0)
       (effects (font (size 1.27 1.27)) hide)
     )
@@
   (symbol (lib_id "power:GND") (at 55.88 67.31 0) (unit 1)
     (in_bom yes) (on_board yes) (fields_autoplaced)
-    (property "Reference" "#PWR050" (id 0) (at 55.88 73.66 0)
+    (property "Reference" "#PWR054" (id 0) (at 55.88 73.66 0)
       (effects (font (size 1.27 1.27)) hide)
     )
@@
   (symbol (lib_id "power:GND") (at 55.88 125.73 0) (unit 1)
     (in_bom yes) (on_board yes) (fields_autoplaced)
-    (property "Reference" "#PWR052" (id 0) (at 55.88 132.08 0)
+    (property "Reference" "#PWR056" (id 0) (at 55.88 132.08 0)
       (effects (font (size 1.27 1.27)) hide)
     )
@@
   (symbol (lib_id "custom_connetors:Conn_01x10_TI30XA") (at 162.56 140.97 0) (unit 2)
     (in_bom yes) (on_board yes)
-    (property "Reference" "J3" (id 0) (at 167.64 139.6999 0)
-      (effects (font (size 1.27 1.27)) (justify left))
-    )
+    (property "Reference" "J7" (id 0) (at 167.64 139.6999 0)
+      (effects (font (size 1.27 1.27)) (justify left))
+    )
