File: calculator_interface/lcd.kicad_sch (KiCad schematic)
At the start: 60 parts, among them J2 Conn_02x20_TI30XA, U10 LM339, U11 74HC165, U12 LM339, U13 LM339, U2 74HC165, U3 LM339, U4 LM339, U5 74HC165, U6 LM339, U7 LM339, U8 74HC165, U9 LM339

Commit message: changed reference voltage circuit to be compatible with voltage regulator
Parts:
- R33, R34: value 100K -> 100R; footprint Resistor_THT:R_Axial_DIN0204_L3.6mm_D1.6mm_P7.62mm_Horizontal -> Resistor_THT:R_Axial_DIN0207_L6.3mm_D2.5mm_P10.16mm_Horizontal
Connections:
- net Comparator reference: now reaches C17.1, R33.2, R34.1, U10.10 (-), U10.4 (-), U10.6 (-), U10.8 (-), U12.10 (-), U12.4 (-), U12.6 (-), U12.8 (-), U13.10 (-), U13.4 (-), U13.6 (-), U13.8 (-), U4.10 (-), U4.4 (-), U4.6 (-), U4.8 (-), U6.10 (-), U6.4 (-), U6.6 (-), U6.8 (-), U7.10 (-), U7.4 (-), U7.6 (-), U7.8 (-), U9.10 (-), U9.4 (-), U9.6 (-), U9.8 (-)
Changed lines of the file:
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@@
+    (effects (font (size 1.27 1.27)) (justify left bottom))
+  )
+  (label "Comparator reference" (at 236.22 68.58 0)
     (effects (font (size 1.27 1.27)) (justify left bottom))
   )
@@
       (effects (font (size 1.27 1.27)) (justify left))
     )
-    (property "Value" "100K" (id 1) (at 238.76 77.4699 0)
-      (effects (font (size 1.27 1.27)) (justify left))
-    )
-    (property "Footprint" "Resistor_THT:R_Axial_DIN0204_L3.6mm_D1.6mm_P7.62mm_Horizontal" (id 2) (at 234.442 76.2 90)
+    (property "Value" "100R" (id 1) (at 238.76 77.4699 0)
+      (effects (font (size 1.27 1.27)) (justify left))
+    )
+    (property "Footprint" "Resistor_THT:R_Axial_DIN0207_L6.3mm_D2.5mm_P10.16mm_Horizontal" (id 2) (at 234.442 76.2 90)
       (effects (font (size 1.27 1.27)) hide)
     )
@@
       (effects (font (size 1.27 1.27)) (justify left))
     )
-    (property "Value" "100K" (id 1) (at 238.76 63.4999 0)
-      (effects (font (size 1.27 1.27)) (justify left))
-    )
-    (property "Footprint" "Resistor_THT:R_Axial_DIN0204_L3.6mm_D1.6mm_P7.62mm_Horizontal" (id 2) (at 234.442 62.23 90)
-      (effects (font (size 1.27 1.27)) hide)
-    )
+    (property "Value" "100R" (id 1) (at 238.76 63.4999 0)
+      (effects (font (size 1.27 1.27)) (justify left))
+    )
+    (property "Footprint" "Resistor_THT:R_Axial_DIN0207_L6.3mm_D2.5mm_P10.16mm_Horizontal" (id 2) (at 234.442 62.23 90)
+      (effects (font (size 1.27 1.27)) hide)
+    )
